File: kicad/Unicycle.kicad_pcb (KiCad board)
At the start: 2 copper layers, 120 x 120 mm, 19 parts, among them IC1 TSR 2 2450, P3 Battery Connector, P4 Safety Switch Connector, P5 Motor Driver Connector, P6 IMU Connector, U1 Teensy4.0

Commit message: update
Parts:
- removed the P1 at (116.0, 102.1)
- removed the P2 at (115.9, 117.7)
- removed P6: IMU Connector, Connector_PinHeader_2.54mm:PinHeader_1x04_P2.54mm_Vertical
- removed U1: Teensy4.0, teensy_foot:Teensy40
- added A3: Pololu LSM6DSO, unicycle_foot:PololuLSM6DSO Text Up, F.Cu at (153.6, 109.8)
- added A4: Teensy 4.0, unicycle_foot:Teensy40 Simple, F.Cu at (152.3, 127.2)
- added J1: HEDS 5500 A, Connector_PinHeader_2.54mm:PinHeader_1x04_P2.54mm_Vertical, F.Cu at (132.5, 147.0)
- added J2: HEDS 5500 A, Connector_PinHeader_2.54mm:PinHeader_1x04_P2.54mm_Vertical, F.Cu at (148.9, 147.2)
- A1, A2: footprint unicycle_foot:Pololu G2 18v17 -> unicycle_foot:Pololu G2 18v17 Text Up
- P1: renamed from P3; footprint Connector_PinHeader_2.54mm:PinHeader_1x02_P2.54mm_Vertical -> Connector_AMASS:AMASS_XT60-F_1x02_P7.20mm_Vertical
- P2: renamed from P4; footprint Connector_PinHeader_2.54mm:PinHeader_1x02_P2.54mm_Vertical -> Connector_AMASS:AMASS_XT60-F_1x02_P7.20mm_Vertical
- P3: renamed from P5; footprint Connector_PinHeader_2.54mm:PinHeader_1x02_P2.54mm_Vertical -> Connector_AMASS:AMASS_XT60-F_1x02_P7.20mm_Vertical
- moved IC1 71.6 mm to (123.8, 127.5)
- moved P3 59.7 mm to (169.9, 97.5), turned to 90 degrees
- moved P1 52.1 mm to (123.8, 107.0), turned to 90 degrees
- moved R3 40.5 mm to (157.5, 141.1), turned to 0 degrees
- moved R1 40.5 mm to (141.0, 141.3), turned to 0 degrees
- moved P2 40.5 mm to (144.5, 88.3), turned to 180 degrees
- moved G*** 36.6 mm to (177.4, 159.4)
- moved R2 34.0 mm to (136.1, 141.4), turned to 180 degrees
- moved R4 33.9 mm to (152.6, 141.0), turned to 180 degrees
- moved H1 29.5 mm to (214.3, 81.7)
- moved H2 26.0 mm to (115.0, 81.0)
- moved A2 20.6 mm to (194.9, 111.2)
- moved H4 11.0 mm to (214.7, 164.7)
- moved A1 5.43 mm to (194.7, 137.7)
- moved H3 1.22 mm to (115.3, 164.7)
Connections:
- A1 pad 2: /DIRP -> DIR_ROLL
- A1 pad 3: /PWMP -> PWM_ROLL
- A2 pad 2: /PWMR -> DIR_PITCH
- A2 pad 3: /DIRR -> PWM_PITCH
- P1 pad 1: +BATT -> GND
- P1 pad 2: GND -> +BATT
- P2 pad 1: +BATT -> VM_LIM
- P2 pad 2: /VM_LIM -> +BATT
- P3 pad 1: /VM_LIM -> GND
- P3 pad 2: GND -> VM_LIM
- R1 pad 2: /AR -> ENC_B_ROLL
- R2 pad 2: /BR -> ENC_A_ROLL
- R3 pad 2: /AP -> ENC_B_PITCH
- R4 pad 2: /BP -> ENC_A_PITCH
Routing:
- net GND: track 49.0 -> 193.5 mm
- net /VM_LIM: track 101.2 -> 0.00 mm
- net /SDA: track 76.8 -> 0.00 mm
- net /SCL: track 71.8 -> 0.00 mm
- net /PWMP: track 61.1 -> 0.00 mm
- net /DIRR: track 54.3 -> 0.00 mm
- net /DIRP: track 49.3 -> 0.00 mm
- net /PWMR: track 47.6 -> 0.00 mm
- net +3.3V: track 99.8 -> 66.8 mm
- net /BP: track 30.4 -> 0.00 mm
- net /AP: track 28.8 -> 0.00 mm
- net +5V: track 101.4 -> 74.5 mm
- net VM_LIM: track 0.00 -> 26.3 mm
- net /BR: track 26.0 -> 0.00 mm
- net /AR: track 24.5 -> 0.00 mm
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Other:
- board size 120 x 120 mm -> 110 x 94 mm
- board text added: "5V"
- board text added: "BATTERY"
- board text added: "MCU"
- board text added: "MOTOR DRIVER PITCH"
- board text added: "MOTOR DRIVER ROLL"
- board text added: "MOTOR POWER"
- board text added: "Nils Axel Andersen, Ulrik Helk DTU Automation & Control"
- board text added: "SAFETY SWITCH"
- board text removed: "BATT IN"
- board text removed: "MOTOR DRV PITCH"
- board text removed: "MOTOR DRV PWR"
- board text removed: "MOTOR DRV ROLL"
- board text removed: "Nils Axel Andersen Ulrik Helk DTU Automation & Control"
- board text removed: "SAFETY SW"

Commit message: Update
Parts:
- added C1: 100nF, Capacitor_SMD:C_0805_2012Metric_Pad1.18x1.45mm_HandSolder, F.Cu at (162.6, 100.9)
- added C10: 1uF, Capacitor_SMD:C_0805_2012Metric_Pad1.18x1.45mm_HandSolder, F.Cu at (117.1, 113.9)
- added C11: 100nF, Capacitor_SMD:C_0805_2012Metric_Pad1.18x1.45mm_HandSolder, F.Cu at (114.6, 113.9)
- added C2: 10uF, Capacitor_SMD:C_1206_3216Metric_Pad1.33x1.80mm_HandSolder, F.Cu at (167.0, 86.0)
- added C3: 4u7F, Capacitor_SMD:C_0805_2012Metric_Pad1.18x1.45mm_HandSolder, F.Cu at (151.1, 100.9)
- added C4: 100nF, Capacitor_SMD:C_0805_2012Metric_Pad1.18x1.45mm_HandSolder, F.Cu at (153.6, 100.9)
- added C5: 1uF, Capacitor_SMD:C_0805_2012Metric_Pad1.18x1.45mm_HandSolder, F.Cu at (154.7, 123.9)
- added C6: 100nF, Capacitor_SMD:C_0805_2012Metric_Pad1.18x1.45mm_HandSolder, F.Cu at (152.2, 123.9)
- added C7: 47uF, Capacitor_SMD:CP_Elec_6.3x3.9, F.Cu at (152.0, 91.3)
- added C8: 1uF, Capacitor_SMD:C_0805_2012Metric_Pad1.18x1.45mm_HandSolder, F.Cu at (117.1, 97.4)
- added C9: 100nF, Capacitor_SMD:C_0805_2012Metric_Pad1.18x1.45mm_HandSolder, F.Cu at (114.6, 97.4)
- added F1: Fuse, Fuse:Fuseholder_Littelfuse_Nano2_154x, F.Cu at (196.5, 66.6)
- added P4: Motor Connector Roll, Connector_AMASS:AMASS_XT60-F_1x02_P7.20mm_Vertical, F.Cu at (222.6, 87.6)
- added Q1: DMP4010SK3Q-13, Package_TO_SOT_SMD:TO-263-2, F.Cu at (179.6, 72.6)
- added Q2: SI2318A-TP, Package_TO_SOT_SMD:SOT-23_Handsoldering, F.Cu at (162.5, 86.0)
- added R10: 220k, Resistor_SMD:R_0805_2012Metric_Pad1.20x1.40mm_HandSolder, F.Cu at (191.1, 72.6)
- added R11: 4.7k, Resistor_SMD:R_0805_2012Metric_Pad1.20x1.40mm_HandSolder, F.Cu at (162.5, 90.5)
- added R5: 10k, Resistor_SMD:R_0805_2012Metric_Pad1.20x1.40mm_HandSolder, F.Cu at (186.7, 127.2)
- added R6: 10k, Resistor_SMD:R_0805_2012Metric_Pad1.20x1.40mm_HandSolder, F.Cu at (213.2, 127.7)
- added R7: 10k, Resistor_SMD:R_0805_2012Metric_Pad1.20x1.40mm_HandSolder, F.Cu at (165.6, 100.9)
- added R8: 47k, Resistor_SMD:R_0805_2012Metric_Pad1.20x1.40mm_HandSolder, F.Cu at (165.0, 97.0)
- added R9: 47k, Resistor_SMD:R_0805_2012Metric_Pad1.20x1.40mm_HandSolder, F.Cu at (165.0, 94.5)
- P1: footprint Connector_AMASS:AMASS_XT60-F_1x02_P7.20mm_Vertical -> Connector_AMASS:AMASS_XT60-M_1x02_P7.20mm_Vertical
- P3: value Motor Driver Connector -> Motor Connector Pitch
- moved H2 112.6 mm to (226.3, 63.7)
- moved H1 101.2 mm to (114.8, 63.3)
- moved G*** 98.0 mm to (81.7, 138.5)
- moved P1 91.1 mm to (208.5, 73.7)
- moved P2 53.1 mm to (197.5, 90.6), turned to 90 degrees
- moved J1 52.1 mm to (120.2, 96.4), turned to 0 degrees
- moved J2 44.9 mm to (120.1, 112.8), turned to 0 degrees
- moved IC1 42.8 mm to (139.7, 87.7), turned to 180 degrees
- moved R2 42.6 mm to (125.8, 100.0), turned to 90 degrees
- moved R1 39.5 mm to (125.8, 104.9), turned to -90 degrees
- moved R3 37.1 mm to (126.1, 121.4), turned to -90 degrees
- moved R4 36.0 mm to (126.2, 116.5), turned to 90 degrees
- moved H4 31.5 mm to (226.5, 135.5)
- moved H3 29.0 mm to (112.8, 135.8)
- moved A1 27.5 mm to (210.9, 115.5), turned to -90 degrees
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Connections:
- A1 pad 4: unconnected-(A1-#SLP-Pad4) -> SLP_ROLL
- A2 pad 4: unconnected-(A2-#SLP-Pad4) -> SLP_PITCH
- A4 pad 12: unconnected-(A4-10_CS_MQSR-Pad12) -> SLP_ROLL
- A4 pad 13: DIR_ROLL -> PWM_ROLL
- A4 pad 14: PWM_ROLL -> DIR_ROLL
- A4 pad 15: PWM_PITCH -> DIR_PITCH
- A4 pad 16: DIR_PITCH -> PWM_PITCH
- A4 pad 17: unconnected-(A4-15_A1_RX3_SPDIF_IN-Pad17) -> SLP_PITCH
- A4 pad 24: unconnected-(A4-22_A8_CTX1-Pad24) -> VBAT_MEAS
- A4 pad 25: unconnected-(A4-23_A9_CRX1_MCLK1-Pad25) -> PWR_ENABLE
- P1 pad 2: +BATT -> Net-(P1-Pin_2)
- P3 pad 1: GND -> OUTB_PITCH
- P3 pad 2: VM_LIM -> OUTA_PITCH
Routing:
- net GND: track 193.5 -> 428.8 mm, vias 0 -> 2
- net SLP_ROLL: track 0.00 -> 87.7 mm
- net PWM_ROLL: track 13.4 -> 86.5 mm
- net DIR_ROLL: track 17.0 -> 88.3 mm
- net +BATT: track 51.6 -> 98.5 mm
- net Net-(Q1-G): track 0.00 -> 42.6 mm, vias 0 -> 2
- net SLP_PITCH: track 0.00 -> 42.6 mm
- net PWM_PITCH: track 12.7 -> 42.8 mm
- net DIR_PITCH: track 15.8 -> 44.7 mm
- net PWR_ENABLE: track 0.00 -> 27.0 mm
- net VBAT_MEAS: track 0.00 -> 25.2 mm
- net VM_LIM: track 26.3 -> 51.0 mm
- net OUTB_ROLL: track 0.00 -> 17.5 mm
- net OUTA_ROLL: track 0.00 -> 16.7 mm
- net OUTA_PITCH: track 0.00 -> 15.5 mm
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Other:
- board size 110 x 94 mm -> 124.2 x 84 mm
