File: kicad/Unicycle.kicad_sch (KiCad schematic)
At the start: 18 parts, among them IC1 TSR 2 2450, P3 Battery Connector, P4 Safety Switch Connector, P5 Motor Driver Connector, P6 IMU Connector, U1 Teensy4.0

Commit message: update
Parts:
- removed P1, P2: ~, Connector_PinHeader_2.54mm:PinHeader_1x04_P2.54mm_Vertical, symbol unicycle:Quad_Connector
- removed P6: IMU Connector, Connector_PinHeader_2.54mm:PinHeader_1x04_P2.54mm_Vertical, symbol unicycle_lib:IMU Connector
- removed U1: Teensy4.0, teensy_foot:Teensy40, symbol teensy_lib:Teensy4.0
- added A3: Pololu LSM6DSO, unicycle_foot:PololuLSM6DSO Text Up, symbol unicycle_lib:Pololu LSM6DSO
- added A4: Teensy 4.0, unicycle_foot:Teensy40 Simple, symbol unicycle_lib:Teensy4.0 Simple
- added J1, J2: HEDS 5500 A, Connector_PinHeader_2.54mm:PinHeader_1x04_P2.54mm_Vertical, symbol Connector_Generic:Conn_01x04
- A1, A2: footprint unicycle_foot:Pololu G2 18v17 -> unicycle_foot:Pololu G2 18v17 Text Up
- P1: renamed from P3; footprint Connector_PinHeader_2.54mm:PinHeader_1x02_P2.54mm_Vertical -> Connector_AMASS:AMASS_XT60-F_1x02_P7.20mm_Vertical; symbol unicycle_lib:Battery Connector -> Connector_Generic:Conn_01x02
- P2: renamed from P4; footprint Connector_PinHeader_2.54mm:PinHeader_1x02_P2.54mm_Vertical -> Connector_AMASS:AMASS_XT60-F_1x02_P7.20mm_Vertical; symbol unicycle_lib:Safety Switch Connector -> Connector_Generic:Conn_01x02
- P3: renamed from P5; footprint Connector_PinHeader_2.54mm:PinHeader_1x02_P2.54mm_Vertical -> Connector_AMASS:AMASS_XT60-F_1x02_P7.20mm_Vertical; symbol unicycle_lib:Motor Driver Connector -> Connector_Generic:Conn_01x02
Connections:
- net +3.3V: now also A3.2 (VIN), A4.26 (3V3)
- net +5V: now also A4.28 (VIN), J1.1 (Pin_1), J2.1 (Pin_1)
- net +BATT: now also P1.2 (Pin_2), P2.2 (Pin_2); no longer P1.1 (+VBAT), P2.1 (+VBAT_IN)
- net GND: now also P1.1 (Pin_1), P3.1 (Pin_1), A3.3 (GND), A4.1 (GND), A4.27 (GND), J1.2 (Pin_2), J2.2 (Pin_2); no longer P1.2 (GND), P3.2 (GND)
- net SCL: now also A3.5 (SCL), A4.21 (19_A5_SCL0)
- net SDA: now also A3.4 (SDA), A4.20 (18_A4_SDA0)
- net VM_LIM: now also P2.1 (Pin_1), P3.2 (Pin_2); no longer P2.2 (+VBAT_OUT), P3.1 (VM_IN)
- net AP renamed ENC_B_PITCH
- net ENC_B_PITCH: now also A4.5 (3_LRCLK2), J2.4 (Pin_4)
- net AR renamed ENC_B_ROLL
- net ENC_B_ROLL: now also A4.3 (1_TX1_CTX2_MISO1), J1.4 (Pin_4)
- net BP renamed ENC_A_PITCH
- net ENC_A_PITCH: now also A4.4 (2_OUT2), J2.3 (Pin_3)
- net BR renamed ENC_A_ROLL
- net ENC_A_ROLL: now also A4.2 (0_RX1_CRX2_CS1), J1.3 (Pin_3)
- net DIRP renamed DIR_ROLL
- net DIR_ROLL: now also A4.13 (11_MOSI_CTX1)
- net DIRR renamed PWM_PITCH
- net PWM_PITCH: now also A4.15 (13_SCK_CRX1_LED)
- net PWMP renamed PWM_ROLL
- net PWM_ROLL: now also A4.14 (12_MISO_MQSL)
- net PWMR renamed DIR_PITCH
- net DIR_PITCH: now also A4.16 (14_A0_TX3_SPDIF_OUT)
- new net SA0: A3.6 (SA0), A4.22 (20_A6_TX5_LRCLK1)
- no-connect marks 41 -> 27
Other:
- note added: "I/O"
- note added: "MCU"
- note added: "MOUNTING"
- note added: "POWER"
- moved on the sheet: A1, A2, H1, H2, H3, H4, IC1, R1, R2, R3, R4

Commit message: Update
Parts:
- added C1, C11, C4, C6, C9: 100nF, Capacitor_SMD:C_0805_2012Metric_Pad1.18x1.45mm_HandSolder, symbol Device:C_Small
- added C10, C5, C8: 1uF, Capacitor_SMD:C_0805_2012Metric_Pad1.18x1.45mm_HandSolder, symbol Device:C_Small
- added C2: 10uF, Capacitor_SMD:C_1206_3216Metric_Pad1.33x1.80mm_HandSolder, symbol Device:C_Small
- added C3: 4u7F, Capacitor_SMD:C_0805_2012Metric_Pad1.18x1.45mm_HandSolder, symbol Device:C_Small
- added C7: 47uF, Capacitor_SMD:CP_Elec_6.3x3.9, symbol Device:C_Polarized_Small
- added F1: Fuse, Fuse:Fuseholder_Littelfuse_Nano2_154x, symbol Device:Fuse
- added J4: Conn_01x07, symbol Connector_Generic:Conn_01x07
- added P4: Motor Connector Roll, Connector_AMASS:AMASS_XT60-F_1x02_P7.20mm_Vertical, symbol Connector_Generic:Conn_01x02
- added Q1: DMP4010SK3Q-13, Package_TO_SOT_SMD:TO-263-2, symbol Device:Q_PMOS_GDS
- added Q2: SI2318A-TP, Package_TO_SOT_SMD:SOT-23_Handsoldering, symbol Device:Q_NMOS_GSD
- added R10: 220k, Resistor_SMD:R_0805_2012Metric_Pad1.20x1.40mm_HandSolder, symbol Device:R
- added R11: 4.7k, Resistor_SMD:R_0805_2012Metric_Pad1.20x1.40mm_HandSolder, symbol Device:R
- added R5, R6, R7: 10k, Resistor_SMD:R_0805_2012Metric_Pad1.20x1.40mm_HandSolder, symbol Device:R
- added R8, R9: 47k, Resistor_SMD:R_0805_2012Metric_Pad1.20x1.40mm_HandSolder, symbol Device:R
- added SW1: SW_Nidec_CAS-120A1, Button_Switch_SMD:Nidec_Copal_CAS-120A, symbol Switch:SW_Nidec_CAS-120A1
- P1: footprint Connector_AMASS:AMASS_XT60-F_1x02_P7.20mm_Vertical -> Connector_AMASS:AMASS_XT60-M_1x02_P7.20mm_Vertical
- P3: value Motor Driver Connector -> Motor Connector Pitch
Connections:
- net +3.3V: now also C5.1, C6.1, J4.2 (Pin_2)
- net +5V: now also C10.1, C11.1, C3.1, C4.1, C8.1, C9.1, J4.1 (Pin_1)
- net +BATT: now also C7.1, Q1.2 (D), R9.1; no longer P1.2 (Pin_2)
- net DIR_PITCH: now also A4.15 (13_SCK_CRX1_LED); no longer A4.16 (14_A0_TX3_SPDIF_OUT)
- net DIR_ROLL: now also A4.14 (12_MISO_MQSL); no longer A4.13 (11_MOSI_CTX1)
- net GND: now also A1.9 (GND_M), A2.9 (GND_M), C1.2, C10.2, C11.2, C2.2, C3.2, C4.2, C5.2, C6.2, C7.2, C8.2, C9.2, J4.3 (Pin_3), Q2.2 (S), R11.2, R5.1, R6.1, R7.2; no longer P3.1 (Pin_1)
- net PWM_PITCH: now also A4.16 (14_A0_TX3_SPDIF_OUT); no longer A4.15 (13_SCK_CRX1_LED)
- net PWM_ROLL: now also A4.13 (11_MOSI_CTX1); no longer A4.14 (12_MISO_MQSL)
- net VM_LIM: now also A1.12 (VM), A2.12 (VM); no longer P3.2 (Pin_2)
- net SLP_ROLL: now reaches A1.4 (#SLP)
- net SLP_ROLL: now also A4.12 (10_CS_MQSR), R6.2
- net SLP_PITCH: now reaches A2.4 (#SLP)
- net SLP_PITCH: now also A4.17 (15_A1_RX3_SPDIF_IN), R5.2
- net IOC: now reaches A4.10 (8_TX2_IN1)
- net IOC: now also J4.6 (Pin_6)
- net IOD: now reaches A4.11 (9_OUT1C)
- net IOD: now also J4.7 (Pin_7)
- net VBAT_MEAS: now reaches A4.24 (22_A8_CTX1)
- net VBAT_MEAS: now also C1.1, R7.1, R8.2
- net PWR_ENABLE: now reaches A4.25 (23_A9_CRX1_MCLK1)
- net PWR_ENABLE: now also Q2.1 (G), R11.1
- net IOA: now reaches A4.8 (6_OUT1D)
- net IOA: now also J4.4 (Pin_4)
- net IOB: now reaches A4.9 (7_RX2_OUT1A)
- net IOB: now also J4.5 (Pin_5)
- new net: R8.1, R9.2
- new net: F1.2, Q1.3 (S), R10.1
- new net: C2.1, Q1.1 (G), Q2.3 (D), R10.2
- new net: F1.1, SW1.3 (A)
- new net: P1.2 (Pin_2), SW1.2 (B)
- new net OUTA_PITCH: A2.11 (OUTA), P3.2 (Pin_2)
- new net OUTA_ROLL: A1.11 (OUTA), P4.2 (Pin_2)
- new net OUTB_PITCH: A2.10 (OUTB), P3.1 (Pin_1)
- new net OUTB_ROLL: A1.10 (OUTB), P4.1 (Pin_1)
- no-connect marks 27 -> 19
Other:
- note added: "26V * R1 / (R1 + R2) = 2.5V R1 = 10k R2 = (26V / 2.5V - 1)*R1 = 94k = 2 * 47k tau = R1*R2/(R1+R2)*C = 0.9 ms"
- note added: "ENCODERS"
- note added: "IMU"
- note added: "MOTOR DRIVERS"
- note removed: "I/O"
- moved on the sheet: A3, A4, H1, H2, H3, H4, IC1, J1, J2, P1, P2, P3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
